File: Micro-Mouse Power Subsystem Final.kicad_sch (KiCad schematic)
At the start: 67 parts, among them J3 USB_C_Receptacle_USB2.0_16P, J4 Battery terminals, J5 Conn_02x16_Odd_Even, Q1 DMP3099L, Q2 2N7002, Q3 DMP3099L, SW1 SW_SPDT, U1 DRV8833PWP, U13 INA219AxD, U2 DRV8833PWP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

Commit message: Add files via upload
updating the schematic
Other:
- note added: "MOSFETS used as high-side load switches for external loads"
- note added: "PD trigger IC negotiates a 9V output from a USB-C source"
- note added: "Pins connecting the power board to motherboard"
- note added: "The INA219 sensor measures real-time battery voltage and current using high-side sensing and I²C communication. Also hooked up to the master switch control power to the entire board."
- moved on the sheet: C14, C16, J3, J5, Q1, Q3, R10, R11, R22, R23, R24, R25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

Commit message: Add files via upload
Other:
- note removed: "MOSFETS used as high-side load switches for external loads"
- note removed: "PD trigger IC negotiates a 9V output from a USB-C source"
- note removed: "Pins connecting the power board to motherboard"
- note removed: "The INA219 sensor measures real-time battery voltage and current using high-side sensing and I²C communication. Also hooked up to the master switch control power to the entire board."
- moved on the sheet: C14, C16, J3, J5, Q1, Q3, R10, R11, R22, R23, R24, R25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

Commit message: Add files via upload
Other:
- note added: "MOSFETS used as high-side load switches for external loads"
- note added: "PD trigger IC negotiates a 9V output from a USB-C source"
- note added: "Pins connecting the power board to motherboard"
- note added: "Set Charging Modes: Controlled by the Processor via Power Submodule pin 13 (Fast Charge Control) 200 mA and 600 mA charging currents by enabling or disabling the fast charge pathway through the MOSFET"
- note added: "Steps down 9V from PD trigger IC (HV) to 5V"
- note added: "The INA219 sensor measures real-time battery voltage and current using high-side sensing and I²C communication. Also hooked up to the master switch control power to the entire board."
- note removed: "Set Charging Modes(jumper pin 2-3 always closed) 200mA-jumper pin 1-2 closed ~600mA(±100mA)-jumper pin 1-2 open"
- moved on the sheet: C14, C16, J3, J5, Q1, Q3, R10, R11, R22, R23, R24, R25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
